Commit message: update add realsense and ouster

File: unitree_ros/robots/go1_description/urdf/go1.urdf (robot description, URDF)
Before this commit: robot go1, 47 links, 46 joints
Links:
- added link ouster_link, mass 1e-5; collision cylinder length=0.05 radius=0.05; visual cylinder length=0.08 radius=0.04
Joints:
- added joint camera_joint: type fixed, parent trunk, child camera_link, origin xyz=0.1481 0 0.16 rpy=0 0 0
- added joint ouster_joint: type fixed, parent trunk, child os_sensor, origin xyz=0.0125 0 0.17 rpy=0 0 0
- added joint ouster_visual_joint: type fixed, parent ouster_joint, child ouster_link, origin xyz=0 0 0 rpy=0 0 0

File: unitree_ros/robots/go1_description/xacro/robot.xacro (robot description, xacro)
@@ -129,3 +129,6 @@
         <origin rpy="0 0 0" xyz="0.05 0 0.08"/>
     </xacro:lidar>
+    <xacro:cps_additions parent="trunk">
+        <!-- <origin rpy="0 0 0" xyz="0.1481 0 0.16"/> -->
+    </xacro:lidar>
 </robot>
