Commit message: update

File: unitree_ros/robots/go1_description/xacro/cps_additions.xacro (robot description, xacro)
@@ -8,5 +8,5 @@
             <xacro:insert_block name="origin"/>
             <origin rpy="0 0 0" xyz="0.1481 0 0.16"/>
-            <parent link="${parent}"/>
+            <parent link="trunk"/>
             <child link="camera_link"/>
         </joint>
@@ -14,5 +14,5 @@
         <joint name="ouster_joint" type="fixed">
             <origin rpy="0 0 0" xyz="0.0125 0 0.17"/>
-            <parent link="${parent}"/>
+            <parent link="trunk"/>
             <child link="os_sensor"/>
         </joint>
