Commit message: update

File: unitree_ros/robots/go1_description/xacro/robot.xacro (robot description, xacro)
@@ -130,6 +130,40 @@
         <origin rpy="0 0 0" xyz="0.05 0 0.08"/>
     </xacro:lidar>
-    <xacro:cps_additions>
-        <!-- <origin rpy="0 0 0" xyz="0.1481 0 0.16"/> -->
-    </xacro:cps_additions>
+    <joint name="camera_joint" type="fixed">
+        <xacro:insert_block name="origin"/>
+        <origin rpy="0 0 0" xyz="0.1481 0 0.16"/>
+        <parent link="trunk"/>
+        <child link="camera_link"/>
+    </joint>
+    <!-- ouster -->
+    <joint name="ouster_joint" type="fixed">
+        <origin rpy="0 0 0" xyz="0.0125 0 0.17"/>
+        <parent link="trunk"/>
+        <child link="os_sensor"/>
+    </joint>
+    <joint name="ouster_visual_joint" type="fixed">
+        <origin rpy="0 0 0" xyz="0 0 0"/>
+        <parent link="ouster_joint"/>
+        <child link="ouster_link"/>
+    </joint>
+    <link name="ouster_link">
+        <collision>
+        <origin rpy="0 0 0" xyz="0 0 0"/>
+        <geometry>
+            <cylinder length="0.05" radius="0.05"/>
+        </geometry>
+        </collision>
+        <visual>
+        <origin rpy="0 0 0" xyz="0 0 0"/>
+        <geometry>
+            <cylinder length="0.08" radius="0.04"/>
+        </geometry>
+        <material name="black"/>
+        </visual>
+        <inertial>
+        <mass value="1e-5"/>
+        <origin rpy="0 0 0" xyz="0 0 0"/>
+        <inertia ixx="1e-6" ixy="0" ixz="0" iyy="1e-6" iyz="0" izz="1e-6"/>
+        </inertial>
+    </link>
 </robot>

Commit message: update

File: unitree_ros/robots/go1_description/xacro/robot.xacro (robot description, xacro)
@@ -130,4 +130,5 @@
         <origin rpy="0 0 0" xyz="0.05 0 0.08"/>
     </xacro:lidar>
+<!--
     <joint name="camera_joint" type="fixed">
         <xacro:insert_block name="origin"/>
@@ -135,5 +136,5 @@
         <parent link="trunk"/>
         <child link="camera_link"/>
-    </joint>
+    </joint> -->
     <!-- ouster -->
     <joint name="ouster_joint" type="fixed">

Commit message: update

File: unitree_ros/robots/go1_description/xacro/robot.xacro (robot description, xacro)
@@ -143,4 +143,6 @@
         <child link="os_sensor"/>
     </joint>
+    <link_name="os_sensor">
+    </link>
     <joint name="ouster_visual_joint" type="fixed">
         <origin rpy="0 0 0" xyz="0 0 0"/>

Commit message: update

File: unitree_ros/robots/go1_description/xacro/robot.xacro (robot description, xacro)
@@ -130,11 +130,11 @@
         <origin rpy="0 0 0" xyz="0.05 0 0.08"/>
     </xacro:lidar>
-<!--
     <joint name="camera_joint" type="fixed">
-        <xacro:insert_block name="origin"/>
         <origin rpy="0 0 0" xyz="0.1481 0 0.16"/>
         <parent link="trunk"/>
         <child link="camera_link"/>
-    </joint> -->
+    </joint>
+    <link_name="camera_link">
+    </link>
     <!-- ouster -->
     <joint name="ouster_joint" type="fixed">

Commit message: update

File: unitree_ros/robots/go1_description/xacro/robot.xacro (robot description, xacro)
@@ -135,5 +135,5 @@
         <child link="camera_link"/>
     </joint>
-    <link_name="camera_link">
+    <link name="camera_link">
     </link>
     <!-- ouster -->
@@ -143,5 +143,5 @@
         <child link="os_sensor"/>
     </joint>
-    <link_name="os_sensor">
+    <link name="os_sensor">
     </link>
     <joint name="ouster_visual_joint" type="fixed">

Commit message: update

File: unitree_ros/robots/go1_description/xacro/robot.xacro (robot description, xacro)
@@ -147,5 +147,5 @@
     <joint name="ouster_visual_joint" type="fixed">
         <origin rpy="0 0 0" xyz="0 0 0"/>
-        <parent link="ouster_joint"/>
+        <parent link="os_sensor"/>
         <child link="ouster_link"/>
     </joint>

Commit message: update

File: unitree_ros/robots/go1_description/xacro/robot.xacro (robot description, xacro)
@@ -130,7 +130,15 @@
         <origin rpy="0 0 0" xyz="0.05 0 0.08"/>
     </xacro:lidar>
+    <joint name="camera_base_joint" type="fixed">
+        <origin rpy="0 0 0" xyz="0.150 0 0.147"/>
+        <parent link="trunk"/>
+        <child link="camera_base"/>
+    </joint>
+    <link name="camera_base">
+    </link>
     <joint name="camera_joint" type="fixed">
-        <origin rpy="0 0 0" xyz="0.1481 0 0.16"/>
-        <parent link="trunk"/>
+    <!-- is in fact the rgb camera position which is offset + 17.5 mm y direction -->
+        <origin rpy="0 0 0" xyz="0 0.0175 0"/>
+        <parent link="camera_base"/>
         <child link="camera_link"/>
     </joint>
@@ -139,5 +147,5 @@
     <!-- ouster -->
     <joint name="ouster_joint" type="fixed">
-        <origin rpy="0 0 0" xyz="0.0125 0 0.17"/>
+        <origin rpy="0 0 0" xyz="0.072 0 0.214"/>
         <parent link="trunk"/>
         <child link="os_sensor"/>
